File: pcb/CRX1.sch (KiCad schematic (older format))
At the start: 141 parts, among them J1 ANT, J2 EXT VFO, J3 Key Line, J4 +12 VDC, J5 Phones, P1 XTAL GND, P2 BFO, P3 VXO, P4 Sidetone, P5 GND, Q1 MMBFJ310, Q10 MMBT4403, Q11 MMBT4401, Q12 MMBT4403, Q13 MMBT4401, Q14 2N7002, Q15 MMBT4401, Q16 MMBT4401, Q17 MMBT4403, Q2 MMBT4401, Q3 MMBFJ310, Q4 BF998, Q5 BF998, Q6 2N7002, Q7 2N7002, Q8 2N7002, Q9 IRLML9301, T1 FT37-43 6T:20T, X1 4.032 MHz, X2 4.032 MHz, X3 4.032 MHz, X4 4.032 MHz, X5 11.059 MHz, X6 11.059 MHz

Commit message: Rev A Production
Parts:
- added C44: 47, symbol C
- added C45: 100n, symbol C
- added D9: LL4148, symbol DIODE
- C30: value 4.7u MLCC -> 1u MLCC
- R19: value 10k -> 4.7k
- R33: value 47 -> 470
Connections:
- net GND: now also R40.1, C45.2
- net at Q14.2 (G), R40.2: now also JP2.2
- net at D4.2 (K), Q6.2 (G), R23.2: now also C45.1
- net at C11.1, C14.1, C19.1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: now also C44.2; no longer L1.2
- net at J3.1, J3.2: now also D9.2 (K); no longer R25.1
- new net: C44.1, L1.2
- new net: D9.1 (A), R25.1
Other:
- moved on the sheet: C3, D1, D2, J1, J3, L1, Q8, R24, R40
